File: ArduinoNanoESP32/KiCad_8.0/KiCad_Arduino_IOTAudioSwitch/KiCad_Arduino_IOTAudioSwitch.kicad_pcb (KiCad board)
At the start: 2 copper layers, 0 parts

Commit message: Created PCB
Parts:
- added A1: Arduino_Nano_ESP32_Socket, PCM_arduino-library:Arduino_Nano_ESP32_Socket, F.Cu at (199.2, 112.9)
- added C1: 0.1 uF, Capacitor_THT:C_Disc_D8.0mm_W2.5mm_P5.00mm, F.Cu at (165.1, 74.8)
- added C10: 1 uF, Capacitor_THT:C_Disc_D8.0mm_W2.5mm_P5.00mm, F.Cu at (163.0, 102.0)
- added C2: 10 uF, Capacitor_THT:CP_Radial_D5.0mm_P2.00mm, F.Cu at (159.9, 74.7)
- added C3: 1 uF, Capacitor_THT:C_Disc_D8.0mm_W2.5mm_P5.00mm, F.Cu at (163.0, 55.0)
- added C4: 1 uF, Capacitor_THT:C_Disc_D8.0mm_W2.5mm_P5.00mm, F.Cu at (163.0, 45.0)
- added C5: 1 uF, Capacitor_THT:C_Disc_D8.0mm_W2.5mm_P5.00mm, F.Cu at (163.0, 71.0)
- added C6: 1 uF, Capacitor_THT:C_Disc_D8.0mm_W2.5mm_P5.00mm, F.Cu at (163.0, 61.0)
- added C7: 1 uF, Capacitor_THT:C_Disc_D8.0mm_W2.5mm_P5.00mm, F.Cu at (163.0, 96.1)
- added C8: 1 uF, Capacitor_THT:C_Disc_D8.0mm_W2.5mm_P5.00mm, F.Cu at (163.0, 86.0)
- added C9: 1 uF, Capacitor_THT:C_Disc_D8.0mm_W2.5mm_P5.00mm, F.Cu at (163.0, 112.0)
- added J1: SJ1-3523NG, Thick 3.5 Jack:SJ13523NG, F.Cu at (205.4, 49.9)
- added J2: SJ1-3523NG, Thick 3.5 Jack:SJ13523NG, F.Cu at (146.3, 50.0)
- added J3: SJ1-3523NG, Thick 3.5 Jack:SJ13523NG, F.Cu at (146.3, 66.0)
- added J4: SJ1-3523NG, Thick 3.5 Jack:SJ13523NG, F.Cu at (146.3, 91.1)
- added J5: SJ1-3523NG, Thick 3.5 Jack:SJ13523NG, F.Cu at (146.3, 107.0)
- added R1: 100 Ohm, Resistor_THT:R_Axial_DIN0207_L6.3mm_D2.5mm_P7.62mm_Horizontal, F.Cu at (185.1, 100.9)
- added R10: 10K Ohm, Resistor_THT:R_Axial_DIN0207_L6.3mm_D2.5mm_P7.62mm_Horizontal, F.Cu at (164.3, 92.8)
- added R11: 10K Ohm, Resistor_THT:R_Axial_DIN0207_L6.3mm_D2.5mm_P7.62mm_Horizontal, F.Cu at (164.3, 89.4)
- added R12: 10K Ohm, Resistor_THT:R_Axial_DIN0207_L6.3mm_D2.5mm_P7.62mm_Horizontal, F.Cu at (164.3, 108.7)
- added R13: 10K Ohm, Resistor_THT:R_Axial_DIN0207_L6.3mm_D2.5mm_P7.62mm_Horizontal, F.Cu at (164.3, 105.4)
- added R2: 100 Ohm, Resistor_THT:R_Axial_DIN0207_L6.3mm_D2.5mm_P7.62mm_Horizontal, F.Cu at (185.1, 104.1)
- added R3: 100 Ohm, Resistor_THT:R_Axial_DIN0207_L6.3mm_D2.5mm_P7.62mm_Horizontal, F.Cu at (185.1, 110.5)
- added R4: 100 Ohm, Resistor_THT:R_Axial_DIN0207_L6.3mm_D2.5mm_P7.62mm_Horizontal, F.Cu at (185.1, 107.3)
- added R5: 0 Ohm, Resistor_THT:R_Axial_DIN0207_L6.3mm_D2.5mm_P7.62mm_Horizontal, F.Cu at (193.5, 66.7)
- added R6: 10K Ohm, Resistor_THT:R_Axial_DIN0207_L6.3mm_D2.5mm_P7.62mm_Horizontal, F.Cu at (164.3, 51.7)
- added R7: 10K Ohm, Resistor_THT:R_Axial_DIN0207_L6.3mm_D2.5mm_P7.62mm_Horizontal, F.Cu at (164.3, 48.4)
- added R8: 10K Ohm, Resistor_THT:R_Axial_DIN0207_L6.3mm_D2.5mm_P7.62mm_Horizontal, F.Cu at (164.3, 67.6)
- added R9: 10K Ohm, Resistor_THT:R_Axial_DIN0207_L6.3mm_D2.5mm_P7.62mm_Horizontal, F.Cu at (164.3, 64.3)
- added U1: CD4052B, 8 Pin DIP Connector:DIPS762W70P254L2032H510Q16N, F.Cu at (168.7, 82.4)
Routing:
- net Net-(U1-Y0): track 0.00 -> 48.2 mm
- net Net-(U1-VDD): track 0.00 -> 48.1 mm
- net Net-(U1-X3): track 0.00 -> 44.9 mm
- net Net-(J1-RING): track 0.00 -> 43.4 mm
- net Net-(J1-TIP): track 0.00 -> 43.0 mm
- net Net-(A1-Pad5V): track 0.00 -> 40.9 mm
- net Net-(U1-B): track 0.00 -> 33.0 mm
- net Net-(U1-X0): track 0.00 -> 30.2 mm
- net Net-(U1-X2): track 0.00 -> 29.9 mm
- net Net-(U1-Y3): track 0.00 -> 29.1 mm
- net Net-(U1-A): track 0.00 -> 28.8 mm
- net Net-(U1-Y1): track 0.00 -> 28.6 mm
- net Net-(U1-INH): track 0.00 -> 27.4 mm
- net Net-(U1-X1): track 0.00 -> 16.2 mm
- net Net-(U1-Y2): track 0.00 -> 13.7 mm
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- added copper zone on B.Cu, net GND
- added copper zone on B.Cu, net GNDA
Other:
- board outline added: 67.3 x 71.1 mm
