File: ArduinoNanoESP32/KiCad_8.0/KiCad_Arduino_IOTAudioSwitch/KiCad_Arduino_IOTAudioSwitch.kicad_sch (KiCad schematic)
At the start: 13 parts, among them J1 SJ1-3523NG, J2 SJ1-3523NG, J3 SJ1-3523NG, J4 SJ1-3523NG, J5 SJ1-3523NG, U1 CD4052B

Commit message: Created PCB
Parts:
- added C10, C3, C4, C5, C6, C7, C8, C9: 1 uF, Capacitor_THT:C_Disc_D8.0mm_W2.5mm_P5.00mm, symbol Device:C
- added C2: 10 uF, Capacitor_THT:CP_Radial_D5.0mm_P2.00mm, symbol Device:C_Polarized
- added R10, R11, R12, R13, R6, R7, R8, R9: 10K Ohm, Resistor_THT:R_Axial_DIN0207_L6.3mm_D2.5mm_P7.62mm_Horizontal, symbol Device:R_US
- C1: footprint (none) -> Capacitor_THT:C_Disc_D8.0mm_W2.5mm_P5.00mm
- J1, J2, J3, J4, J5: footprint SJ13523NG -> Thick 3.5 Jack:SJ13523NG
- R1, R2, R3, R4, R5: footprint (none) -> Resistor_THT:R_Axial_DIN0207_L6.3mm_D2.5mm_P7.62mm_Horizontal
- U1: footprint (none) -> 8 Pin DIP Connector:DIPS762W70P254L2032H510Q16N
Connections:
- net GNDA: now also C2.2, R10.2, R11.2, R12.2, R13.2, R6.2, R7.2, R8.2, R9.2
- net at U1.1 (Y0): now also C4.1, R7.1; no longer J2.3 (RING)
- net at U1.11 (X3): now also C9.1, R12.1; no longer J5.2 (TIP)
- net at U1.12 (X0): now also C3.1, R6.1; no longer J2.2 (TIP)
- net at U1.14 (X1): now also C5.1, R8.1; no longer J3.2 (TIP)
- net at U1.15 (X2): now also C7.1, R10.1; no longer J4.2 (TIP)
- net at C1.1, R3.2, U1.16 (VDD): now also C2.1
- net at U1.2 (Y2): now also C8.1, R11.1; no longer J4.3 (RING)
- net at U1.4 (Y3): now also C10.1, R13.1; no longer J5.3 (RING)
- net at U1.5 (Y1): now also C6.1, R9.1; no longer J3.3 (RING)
- net at A1.D10: now also R2.1
- net at A1.D11 (D11_MOSI): now also R4.1
- net at A1.D2: no longer R1.1
- net at A1.D3: no longer R2.1
- net at A1.D4: no longer R4.1
- net at A1.D9: now also R1.1
- new net: C9.2, J5.2 (TIP)
- new net: C10.2, J5.3 (RING)
- new net: C5.2, J3.2 (TIP)
- new net: C6.2, J3.3 (RING)
- new net: C4.2, J2.3 (RING)
- new net: C8.2, J4.3 (RING)
- new net: C3.2, J2.2 (TIP)
- new net: C7.2, J4.2 (TIP)
Other:
- moved on the sheet: J2
